File: KiCAD/299Clock.kicad_sch (KiCad schematic)
At the start: 30 parts, among them SW1 PEC11R, U1 RPi Pico, U2 RDA5807M, U3 LM386

Commit message: Added test points to PCB
Parts:
- added TEST1, TEST2: Conn_01x01, TestPoint:TestPoint_Pad_1.5x1.5mm, symbol Connector_Generic:Conn_01x01
Connections:
- net at C1.1, D2.1 (K), R3.1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: now also TEST1.1 (Pin_1)
- net at C4.1, C5.1, U3.5: now also TEST2.1 (Pin_1)
Changed lines of the file:
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@@
+    (stroke (width 0) (type default) (color 0 0 0 0))
+  )
+  (wire (pts (xy 228.6 71.12) (xy 228.6 73.66))
     (stroke (width 0) (type default) (color 0 0 0 0))
   )
@@
   )
   (wire (pts (xy 213.36 109.22) (xy 213.36 81.28))
+    (stroke (width 0) (type default) (color 0 0 0 0))
+  )
+  (wire (pts (xy 179.07 68.58) (xy 179.07 71.12))
     (stroke (width 0) (type default) (color 0 0 0 0))
   )
@@
     (pin "1")
     (pin "2")
+  )
+  (symbol (lib_id "Connector_Generic:Conn_01x01") (at 179.07 63.5 90) (unit 1)
+    (in_bom yes) (on_board yes)
+    (property "Reference" "TEST1" (id 0) (at 171.45 63.5 90)
+      (effects (font (size 1.27 1.27)) (justify right))
+    )
+    (property "Value" "Conn_01x01" (id 1) (at 181.61 64.7699 90)
+      (effects (font (size 1.27 1.27)) (justify right) hide)
+    )
+    (property "Footprint" "TestPoint:TestPoint_Pad_1.5x1.5mm" (id 2) (at 179.07 63.5 0)
+      (effects (font (size 1.27 1.27)) hide)
+    )
+    (property "Datasheet" "~" (id 3) (at 179.07 63.5 0)
+      (effects (font (size 1.27 1.27)) hide)
+    )
+    (pin "1")
   )
   (symbol (lib_id "Amplifier_Audio:LM386") (at 215.9 73.66 0) (unit 1)
@@
     (pin "1")
     (pin "2")
+  )
+  (symbol (lib_id "Connector_Generic:Conn_01x01") (at 228.6 66.04 90) (unit 1)
+    (in_bom yes) (on_board yes) (fields_autoplaced)
+    (property "Reference" "TEST2" (id 0) (at 231.14 66.0399 90)
+      (effects (font (size 1.27 1.27)) (justify right))
+    )
+    (property "Value" "Conn_01x01" (id 1) (at 231.14 67.3099 90)
+      (effects (font (size 1.27 1.27)) (justify right) hide)
+    )
+    (property "Footprint" "TestPoint:TestPoint_Pad_1.5x1.5mm" (id 2) (at 228.6 66.04 0)
+      (effects (font (size 1.27 1.27)) hide)
+    )
+    (property "Datasheet" "~" (id 3) (at 228.6 66.04 0)
+      (effects (font (size 1.27 1.27)) hide)
+    )
+    (pin "1")
   )
   (symbol (lib_id "Device:R_US") (at 27.94 143.51 90) (unit 1)
@@
       (reference "SW1") (unit 1) (value "PEC11R") (footprint "Connector_PinHeader_2.54mm:PinHeader_1x05_P2.54mm_Vertical")
     )
+    (path "/8ad63974-f1bb-4e6e-98d3-73d73f9a7e77"
+      (reference "TEST1") (unit 1) (value "Conn_01x01") (footprint "TestPoint:TestPoint_Pad_1.5x1.5mm")
+    )
+    (path "/9771467d-0ba1-49a8-9edf-7d9ec8766cc8"
+      (reference "TEST2") (unit 1) (value "Conn_01x01") (footprint "TestPoint:TestPoint_Pad_1.5x1.5mm")
+    )
     (path "/e5998a09-fd11-4bd9-9f32-af02ea1eafe1"

Commit message: Finished traces, routed sw, add ground planes
Connections:
- net GND: now reaches C2.2, C3.2, C6.2, C7.2, DISP1.1 (VSS/GND), H1.1, H2.1, H3.1, H4.1, LS1.2, R5.2, R6.2, SW1.C, U1.13 (GND), U1.18 (GND), U1.23 (GND), U1.28 (GND), U1.3 (GND), U1.33 (GND), U1.38 (GND), U1.8 (GND), U2.6 (GND), U3.2 (-), U3.4 (GND)
Changed lines of the file:
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@@
   (junction (at 58.42 109.22) (diameter 0) (color 0 0 0 0)
+  )
+  (junction (at 40.64 109.22) (diameter 0) (color 0 0 0 0)
   )
   (junction (at 228.6 109.22) (diameter 0) (color 0 0 0 0)
@@
   )
   (wire (pts (xy 20.32 143.51) (xy 24.13 143.51))
+    (stroke (width 0) (type default) (color 0 0 0 0))
+  )
+  (wire (pts (xy 38.1 109.22) (xy 40.64 109.22))
     (stroke (width 0) (type default) (color 0 0 0 0))
   )
@@
     (pin "9")
   )
+  (symbol (lib_id "power:GND") (at 38.1 109.22 0) (unit 1)
+    (in_bom yes) (on_board yes) (fields_autoplaced)
+    (property "Reference" "#PWR0101" (id 0) (at 38.1 115.57 0)
+      (effects (font (size 1.27 1.27)) hide)
+    )
+    (property "Value" "GND" (id 1) (at 38.1 114.3 0))
+    (property "Footprint" "" (id 2) (at 38.1 109.22 0)
+      (effects (font (size 1.27 1.27)) hide)
+    )
+    (property "Datasheet" "" (id 3) (at 38.1 109.22 0)
+      (effects (font (size 1.27 1.27)) hide)
+    )
+    (pin "1")
+  )
   (symbol (lib_id "Device:R_US") (at 228.6 97.79 0) (unit 1)
     (in_bom yes) (on_board yes) (fields_autoplaced)
@@
   )
   (symbol_instances
+    (path "/e93cb603-50eb-4921-a16b-0acd5e08dd38"
+      (reference "#PWR0101") (unit 1) (value "GND") (footprint "")
+    )
     (path "/391d4315-d7a3-4cf1-829c-d16aea5dab89"
       (reference "AE1") (unit 1) (value "Antenna") (footprint "Connector_Wire:SolderWire-0.1sqmm_1x01_D0.4mm_OD1mm")
