File: KiCAD/299Clock.kicad_sch (KiCad schematic)
At the start: 32 parts, among them SW1 PEC11R, U1 RPi Pico, U2 RDA5807M, U3 LM386

Commit message: revision of PCB and exported gerber
Parts:
- removed C6, C7: 10n, Capacitor_THT:C_Rect_L7.0mm_W2.5mm_P5.00mm, symbol Device:C
- removed R10, R7, R8, R9: 10k, Resistor_THT:R_Axial_DIN0207_L6.3mm_D2.5mm_P10.16mm_Horizontal, symbol Device:R_US
- removed TEST1, TEST2: Conn_01x01, TestPoint:TestPoint_Pad_1.5x1.5mm, symbol Connector_Generic:Conn_01x01
- added J1: 3V3, Connector_Wire:SolderWire-0.1sqmm_1x01_D0.4mm_OD1mm, symbol Connector:Conn_01x01_Male
- added J2: GND, Connector_Wire:SolderWire-0.1sqmm_1x01_D0.4mm_OD1mm, symbol Connector:Conn_01x01_Male
- R1, R2, R3, R4, R5, R6: footprint Resistor_THT:R_Axial_DIN0207_L6.3mm_D2.5mm_P10.16mm_Horizontal -> Resistor_THT:R_Axial_DIN0207_L6.3mm_D2.5mm_P7.62mm_Horizontal
Connections:
- net GND: now also J2.1 (Pin_1); no longer SW1.C
- net at DISP1.2 (VDD), R1.1, R2.1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: now also SW1.C, J1.1 (Pin_1)
- net at SW1.A: now also U1.19 (GP14)
- net at SW1.B: now also U1.17 (GP13)
